File: riocore/plugins/i2c/kicad/i2c/i2c.kicad_pcb (KiCad board)
At the start: 2 copper layers, 13.5 x 24.5 mm, 8 parts, among them U2 ISO1540

Commit message: i2c: kicad: fixes
Connections:
- net 3v3 renamed +3.3V
- net gnd renamed GND
- net m1 renamed /scl
- net m3 renamed /sda

Commit message: kicad: get power-signals
Connections:
- R2 pad 2: +3.3V -> 3V3
- R3 pad 2: +3.3V -> 3V3
- U2 pad 1: +3.3V -> 3V3
Changed lines of the file:
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@@
 	(net 7 "/sda")
 	(net 8 "/scl")
+	(net 9 "3V3")
 	(footprint "Resistor_SMD:R_0805_2012Metric_Pad1.20x1.40mm_HandSolder"
 		(layer "F.Cu")
@@
 			)
 		)
-		(property "Datasheet" ""
+		(property "Datasheet" "~"
 			(at 0 0 0)
 			(layer "F.Fab")
@@
 			(layers "F.Cu" "F.Mask" "F.Paste")
 			(roundrect_rratio 0.25)
-			(net 6 "+3.3V")
+			(net 9 "3V3")
 			(pinfunction "VCC1")
 			(pintype "power_in")
@@
 			)
 		)
-		(property "Datasheet" ""
+		(property "Datasheet" "~"
 			(at 0 0 90)
 			(layer "F.Fab")
@@
 			)
 		)
-		(property "Datasheet" ""
+		(property "Datasheet" "~"
 			(at 0 0 0)
 			(layer "F.Fab")
@@
 			(layers "F.Cu" "F.Mask" "F.Paste")
 			(roundrect_rratio 0.208333)
-			(net 6 "+3.3V")
+			(net 9 "3V3")
 			(pintype "passive")
 		)
@@
 			)
 		)
-		(property "Datasheet" ""
+		(property "Datasheet" "~"
 			(at 0 0 0)
 			(layer "F.Fab")
@@
 			)
 		)
-		(property "Datasheet" ""
+		(property "Datasheet" "~"
 			(at 0 0 90)
 			(layer "F.Fab")
@@
 			)
 		)
-		(property "Datasheet" ""
+		(property "Datasheet" "~"
 			(at 0 0 0)
 			(layer "F.Fab")
@@
 			)
 		)
-		(property "Datasheet" ""
+		(property "Datasheet" "~"
 			(at 0 0 0)
 			(layer "F.Fab")
@@
 			(layers "F.Cu" "F.Mask" "F.Paste")
 			(roundrect_rratio 0.208333)
-			(net 6 "+3.3V")
+			(net 9 "3V3")
 			(pintype "passive")
 		)
