File: riocore/plugins/w5500/kicad/w5500-module/w5500-module.kicad_pcb (KiCad board)
At the start: 2 copper layers, 23.5 x 24.5 mm, 2 parts, among them J15 Conn_01x06, J16 Conn_01x06

Commit message: kicad: recover positions
Connections:
- net /spi_cs renamed /sel
- net /spi_miso renamed /miso
- net /spi_mosi renamed /mosi
- net /spi_sclk renamed /sclk
Changed lines of the file:
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@@
 	(net 2 "gnd")
 	(net 3 "unconnected-(J15-Pin_3-Pad3)")
-	(net 4 "/spi_miso")
+	(net 4 "/miso")
 	(net 5 "3v3")
-	(net 6 "/spi_sclk")
-	(net 7 "/spi_cs")
+	(net 6 "/sclk")
+	(net 7 "/sel")
 	(net 8 "unconnected-(J16-Pin_6-Pad6)")
-	(net 9 "/spi_mosi")
+	(net 9 "/mosi")
 	(footprint "Connector_PinSocket_2.54mm:PinSocket_1x06_P2.54mm_Vertical"
 		(layer "F.Cu")
@@
 			(layers "*.Cu" "*.Mask")
 			(remove_unused_layers no)
-			(net 9 "/spi_mosi")
+			(net 9 "/mosi")
 			(pinfunction "Pin_3")
 			(pintype "passive")
@@
 			(layers "*.Cu" "*.Mask")
 			(remove_unused_layers no)
-			(net 6 "/spi_sclk")
+			(net 6 "/sclk")
 			(pinfunction "Pin_4")
 			(pintype "passive")
@@
 			(layers "*.Cu" "*.Mask")
 			(remove_unused_layers no)
-			(net 7 "/spi_cs")
+			(net 7 "/sel")
 			(pinfunction "Pin_5")
 			(pintype "passive")
@@
 			(layers "*.Cu" "*.Mask")
 			(remove_unused_layers no)
-			(net 4 "/spi_miso")
+			(net 4 "/miso")
 			(pinfunction "Pin_1")
 			(pintype "passive")

Commit message: kicad: get power-signals
Connections:
- net 3v3 renamed +3V3
- net gnd renamed GND
Changed lines of the file:
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@@
 	(net 0 "")
 	(net 1 "unconnected-(J15-Pin_2-Pad2)")
-	(net 2 "gnd")
+	(net 2 "GND")
 	(net 3 "unconnected-(J15-Pin_3-Pad3)")
 	(net 4 "/miso")
-	(net 5 "3v3")
+	(net 5 "+3V3")
 	(net 6 "/sclk")
 	(net 7 "/sel")
@@
 			)
 		)
-		(property "Datasheet" ""
+		(property "Datasheet" "~"
 			(at 0 0 90)
 			(layer "F.Fab")
@@
 			(layers "*.Cu" "*.Mask")
 			(remove_unused_layers no)
-			(net 2 "gnd")
+			(net 2 "GND")
 			(pinfunction "Pin_1")
 			(pintype "passive")
@@
 			(layers "*.Cu" "*.Mask")
 			(remove_unused_layers no)
-			(net 2 "gnd")
+			(net 2 "GND")
 			(pinfunction "Pin_2")
 			(pintype "passive")
@@
 			)
 		)
-		(property "Datasheet" ""
+		(property "Datasheet" "~"
 			(at 0 0 90)
 			(layer "F.Fab")
@@
 			(layers "*.Cu" "*.Mask")
 			(remove_unused_layers no)
-			(net 5 "3v3")
+			(net 5 "+3V3")
 			(pinfunction "Pin_4")
 			(pintype "passive")
@@
 			(layers "*.Cu" "*.Mask")
 			(remove_unused_layers no)
-			(net 5 "3v3")
+			(net 5 "+3V3")
 			(pinfunction "Pin_5")
 			(pintype "passive")
@@
 			(layers "*.Cu" "*.Mask")
 			(remove_unused_layers no)
-			(net 2 "gnd")
+			(net 2 "GND")
 			(pinfunction "Pin_6")
 			(pintype "passive")
@@
 	)
 	(gr_line
+		(start 171.5 88.5)
+		(end 171.5 101.5)
+		(stroke
+			(width 0.1)
+			(type default)
+		)
+		(layer "F.SilkS")
+	)
+	(gr_line
 		(start 171.5 101.5)
 		(end 153.5 101.5)
 		(stroke
 			(width 0.1)
-			(type default)
-		)
-		(layer "F.SilkS")
-	)
-	(gr_line
-		(start 171.5 88.5)
-		(end 171.5 101.5)
-		(stroke
-			(width 0.1)
