File: riocore/plugins/bitin/kicad/optoin/optoin.kicad_pcb (KiCad board)
At the start: 2 copper layers, 13 x 22.5 mm, 6 parts, among them J1 opto_in, U1 LTV-817S

Commit message: generator: new top secret feature :)
Connections:
- net /IN renamed /bit
Changed lines of the file:
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@@
 	(net 3 "F_GND")
 	(net 4 "gnd")
-	(net 5 "/IN")
+	(net 5 "/bit")
 	(net 6 "F_12V")
 	(net 7 "Net-(J1-Pad2)")
@@
 			)
 		)
-		(property "Datasheet" ""
+		(property "Datasheet" "~"
 			(at 0 0 0)
 			(layer "F.Fab")
@@
 			(layers "F.Cu" "F.Mask" "F.Paste")
 			(roundrect_rratio 0.222222)
-			(net 5 "/IN")
+			(net 5 "/bit")
 			(pintype "passive")
 		)
@@
 			)
 		)
-		(property "Datasheet" ""
+		(property "Datasheet" "~"
 			(at 0 0 0)
 			(layer "F.Fab")
@@
 			)
 		)
-		(property "Datasheet" ""
+		(property "Datasheet" "~"
 			(at 0 0 90)
 			(layer "F.Fab")
@@
 			(layers "F.Cu" "F.Mask" "F.Paste")
 			(roundrect_rratio 0.25)
-			(net 5 "/IN")
+			(net 5 "/bit")
 			(pinfunction "K")
 			(pintype "passive")
@@
 			)
 		)
-		(property "Datasheet" ""
+		(property "Datasheet" "~"
 			(at 0 0 0)
 			(layer "F.Fab")
@@
 			(layers "F.Cu" "F.Mask" "F.Paste")
 			(roundrect_rratio 0.140449)
-			(net 5 "/IN")
-			(pintype "passive")
-		)
+			(net 5 "/bit")
+			(pintype "passive")
+		)

Commit message: kicad: get power-signals
Connections:
- net 3v3 renamed +3V3
- net F_12V renamed +24V
- net gnd renamed GND
Changed lines of the file:
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@@
 	)
 	(net 0 "")
-	(net 1 "3v3")
+	(net 1 "+24V")
 	(net 2 "Net-(R85-Pad1)")
 	(net 3 "F_GND")
-	(net 4 "gnd")
+	(net 4 "+3V3")
 	(net 5 "/bit")
-	(net 6 "F_12V")
+	(net 6 "GND")
 	(net 7 "Net-(J1-Pad2)")
 	(net 8 "Net-(D1-A)")
@@
 			(layers "F.Cu" "F.Mask" "F.Paste")
 			(roundrect_rratio 0.222222)
-			(net 1 "3v3")
+			(net 4 "+3V3")
 			(pintype "passive")
 		)
@@
 			(layers "F.Cu" "F.Mask" "F.Paste")
 			(roundrect_rratio 0.222222)
-			(net 1 "3v3")
+			(net 4 "+3V3")
 			(pintype "passive")
 		)
@@
 			(layers "*.Cu" "*.Mask")
 			(remove_unused_layers no)
-			(net 6 "F_12V")
+			(net 1 "+24V")
 			(pintype "passive")
 			(solder_mask_margin 0.102)
@@
 			(layers "F.Cu" "F.Mask" "F.Paste")
 			(roundrect_rratio 0.140449)
-			(net 4 "gnd")
+			(net 6 "GND")
 			(pintype "passive")
 		)
@@
 		(fill no)
 		(layer "Edge.Cuts")
-	)
-	(segment
-		(start 127.425 86.5)
-		(end 127.425 84)
-		(width 0.2)
-		(layer "F.Cu")
-		(net 1)
 	)
 	(segment
@@
 	)
 	(segment
+		(start 127.425 86.5)
+		(end 127.425 84)
+		(width 0.2)
+		(layer "F.Cu")
+		(net 4)
+	)
+	(segment
