File: riocore/plugins/bitout/kicad/transistor/transistor.kicad_pcb (KiCad board)
At the start: 2 copper layers, 12.8 x 17.1 mm, 5 parts, among them J1 bit_out, Q1 BC817

Commit message: kicad: stepstick module
Connections:
- net 3v3 renamed +3V3
- net 5V renamed +5V
- net gnd renamed GND
Changed lines of the file:
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@@
 	)
 	(net 0 "")
-	(net 1 "3v3")
+	(net 1 "+5V")
 	(net 2 "Net-(D1-K)")
-	(net 3 "5V")
-	(net 4 "gnd")
+	(net 3 "GND")
+	(net 4 "+3V3")
 	(net 5 "/bit")
 	(net 6 "Net-(Q1-B)")
@@
 			)
 		)
-		(property "Datasheet" ""
+		(property "Datasheet" "~"
 			(at 0 0 0)
 			(layer "F.Fab")
@@
 			(layers "F.Cu" "F.Mask" "F.Paste")
 			(roundrect_rratio 0.222222)
-			(net 1 "3v3")
+			(net 4 "+3V3")
 			(pintype "passive")
 		)
@@
 			(layers "*.Cu" "*.Mask")
 			(remove_unused_layers no)
-			(net 3 "5V")
+			(net 1 "+5V")
 			(pintype "passive")
 			(solder_mask_margin 0.102)
@@
 			(layers "*.Cu" "*.Mask")
 			(remove_unused_layers no)
-			(net 4 "gnd")
+			(net 3 "GND")
 			(pintype "passive")
 			(solder_mask_margin 0.102)
@@
 			(layers "F.Cu" "F.Mask" "F.Paste")
 			(roundrect_rratio 0.25)
-			(net 4 "gnd")
+			(net 3 "GND")
 			(pinfunction "E")
 			(pintype "passive")
@@
 			)
 		)
-		(property "Datasheet" ""
+		(property "Datasheet" "~"
 			(at 0 0 0)
 			(layer "F.Fab")
@@
 			)
 		)
-		(property "Datasheet" ""
+		(property "Datasheet" "~"
 			(at 0 0 90)
 			(layer "F.Fab")
@@
 		(width 0.2)
 		(layer "F.Cu")
-		(net 4)
+		(net 3)
 	)
 	(segment
@@
 		(width 0.2)
 		(layer "F.Cu")
-		(net 4)
+		(net 3)
 	)
 	(segment
