File: riocore/plugins/satuart/kicad/rs422-master/rs422-master.kicad_pcb (KiCad board)
At the start: 2 copper layers, 19.8 x 33.5 mm, 3 parts, among them J9 RJ45, U17 ADuM1201BR, U18 ADM3488ExR

Commit message: generator: kicad: some fixes
Connections:
- net /RX renamed /rx
- net /TX renamed /tx
Changed lines of the file:
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@@
 	(net 8 "Net-(U17-VIA)")
 	(net 9 "+3V3")
-	(net 10 "/TX")
+	(net 10 "/tx")
 	(net 11 "Net-(U17-VDD2)")
-	(net 12 "/RX")
+	(net 12 "/rx")
 	(net 13 "GND")
 	(footprint "Connector_RJ:RJ45_Amphenol_RJHSE5380"
@@
 			(layers "F.Cu" "F.Mask" "F.Paste")
 			(roundrect_rratio 0.25)
-			(net 12 "/RX")
+			(net 12 "/rx")
 			(pinfunction "VOA")
 			(pintype "output")
@@
 			(layers "F.Cu" "F.Mask" "F.Paste")
 			(roundrect_rratio 0.25)
-			(net 10 "/TX")
+			(net 10 "/tx")
 			(pinfunction "VIB")
 			(pintype "input")

Commit message: kicad: module selection / some fixes
Connections:
- net Net-(J9-Pad4) renamed F_24V
- net Net-(U17-GND2) renamed F_GND
- net Net-(U17-VDD2) renamed F_5V
Changed lines of the file:
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@@
 	(net 0 "")
 	(net 1 "Net-(U18-A)")
-	(net 2 "Net-(J9-Pad4)")
+	(net 2 "F_24V")
 	(net 3 "Net-(U18-Z)")
 	(net 4 "Net-(U18-Y)")
 	(net 5 "Net-(U18-B)")
-	(net 6 "Net-(U17-GND2)")
+	(net 6 "F_GND")
 	(net 7 "Net-(U17-VOB)")
 	(net 8 "Net-(U17-VIA)")
 	(net 9 "+3V3")
 	(net 10 "/tx")
-	(net 11 "Net-(U17-VDD2)")
+	(net 11 "F_5V")
 	(net 12 "/rx")
 	(net 13 "GND")
@@
 		(tags "RJ45 8p8c ethernet cat5")
 		(property "Reference" "J9"
-			(at 3.56 -9.5 0)
+			(at -0.135 -6.075 0)
 			(layer "F.SilkS")
 			(effects
@@
 			)
 		)
-		(property "Datasheet" "~"
+		(property "Datasheet" ""
 			(at 0 0 0)
 			(unlocked yes)
@@
 			(layers "*.Cu" "*.Mask")
 			(remove_unused_layers no)
-			(net 6 "Net-(U17-GND2)")
+			(net 6 "F_GND")
 			(pintype "passive")
 		)
@@
 			(layers "*.Cu" "*.Mask")
 			(remove_unused_layers no)
-			(net 2 "Net-(J9-Pad4)")
+			(net 2 "F_24V")
 			(pintype "passive")
 		)
@@
 			(layers "*.Cu" "*.Mask")
 			(remove_unused_layers no)
-			(net 2 "Net-(J9-Pad4)")
+			(net 2 "F_24V")
 			(pintype "passive")
 		)
@@
 			(layers "*.Cu" "*.Mask")
 			(remove_unused_layers no)
-			(net 6 "Net-(U17-GND2)")
+			(net 6 "F_GND")
 			(pintype "passive")
 		)
@@
 			(layers "F.Cu" "F.Mask" "F.Paste")
 			(roundrect_rratio 0.25)
-			(net 11 "Net-(U17-VDD2)")
+			(net 11 "F_5V")
 			(pinfunction "VCC")
 			(pintype "power_in")
@@
 			(layers "F.Cu" "F.Mask" "F.Paste")
 			(roundrect_rratio 0.25)
-			(net 6 "Net-(U17-GND2)")
+			(net 6 "F_GND")
 			(pinfunction "GND")
 			(pintype "power_in")
@@
 			(layers "F.Cu" "F.Mask" "F.Paste")
 			(roundrect_rratio 0.25)
-			(net 6 "Net-(U17-GND2)")
+			(net 6 "F_GND")
 			(pinfunction "GND2")
 			(pintype "power_in")
@@
 			(layers "F.Cu" "F.Mask" "F.Paste")
 			(roundrect_rratio 0.25)
-			(net 11 "Net-(U17-VDD2)")
+			(net 11 "F_5V")
 			(pinfunction "VDD2")
 			(pintype "power_in")
