File: riocore/plugins/satuart/kicad/rs422-master/rs422-master.kicad_sch (KiCad schematic)
At the start: 3 parts, among them J9 RJ45, U17 ADuM1201BR, U18 ADM3488ExR

Commit message: generator: kicad: some fixes
Connections:
- net RX renamed rx
- net TX renamed tx
Changed lines of the file:
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@@
 		)
 	)
-	(hierarchical_label "RX"
+	(hierarchical_label "rx"
 		(shape input)
 		(at 106.68 93.98 180)
@@
 		)
 	)
-	(hierarchical_label "TX"
+	(hierarchical_label "tx"
 		(shape input)
 		(at 106.68 99.06 180)

Commit message: kicad: module selection / some fixes
Connections:
- net F_GND: now reaches J9.3, J9.6, U17.5 (GND2), U18.4 (GND)
- net F_5V: now reaches U17.8 (VDD2), U18.1 (VCC)
- net F_24V: now reaches J9.4, J9.5
Changed lines of the file:
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@@
+	(wire
+		(pts
+			(xy 99.06 93.98) (xy 106.68 93.98)
+		)
+		(stroke
+			(width 0)
+			(type default)
+		)
+	)
 	(wire
 		(pts
@@
 		(pts
 			(xy 170.18 92.71) (xy 170.18 100.33)
+		)
+		(stroke
+			(width 0)
+			(type default)
+		)
+	)
+	(wire
+		(pts
+			(xy 99.06 99.06) (xy 106.68 99.06)
 		)
 		(stroke
@@
 	(hierarchical_label "rx"
 		(shape input)
-		(at 106.68 93.98 180)
+		(at 99.06 93.98 180)
 		(effects
 			(font
@@
 	(hierarchical_label "tx"
 		(shape input)
-		(at 106.68 99.06 180)
+		(at 99.06 99.06 180)
 		(effects
 			(font
@@
 			)
 			(justify right)
+		)
+	)
+	(symbol
+		(lib_id "power:+3V3")
+		(at 172.72 73.66 0)
+		(unit 1)
+		(exclude_from_sim no)
+		(in_bom yes)
+		(on_board yes)
+		(dnp no)
+		(fields_autoplaced yes)
+		(property "Reference" "#PWR01"
+			(at 172.72 77.47 0)
+			(effects
+				(font
+					(size 1.27 1.27)
+				)
+				(hide yes)
+			)
+		)
+		(property "Value" "F_24V"
+			(at 172.72 68.58 0)
+			(effects
+				(font
+					(size 1.27 1.27)
+				)
+			)
+		)
+		(property "Footprint" ""
+			(at 172.72 73.66 0)
+			(effects
+				(font
+					(size 1.27 1.27)
+				)
+				(hide yes)
+			)
+		)
+		(property "Datasheet" ""
+			(at 172.72 73.66 0)
+			(effects
+				(font
+					(size 1.27 1.27)
+				)
+				(hide yes)
+			)
+		)
+		(property "Description" "Power symbol creates a global label with name \"+3V3\""
+			(at 172.72 73.66 0)
+			(effects
+				(font
+					(size 1.27 1.27)
+				)
+				(hide yes)
+			)
+		)
+		(pin "1"
+		)
+		(instances
+			(project "rs422-master"
+				(path "/a73692ab-48b2-4aab-bf01-a614ece6b97e"
+					(reference "#PWR01")
+					(unit 1)
+				)
+			)
 		)
 	)
@@
 	)
 	(symbol
+		(lib_id "power:GND")
+		(at 151.13 111.76 0)
+		(unit 1)
+		(exclude_from_sim no)
+		(in_bom yes)
+		(on_board yes)
+		(dnp no)
+		(property "Reference" "#PWR03"
+			(at 151.13 118.11 0)
+			(effects
+				(font
+					(size 1.27 1.27)
+				)
+				(hide yes)
+			)
+		)
+		(property "Value" "F_GND"
+			(at 154.686 114.046 0)
+			(effects
+				(font
+					(size 1.27 1.27)
+				)
+			)
+		)
+		(property "Footprint" ""
+			(at 151.13 111.76 0)
+			(effects
+				(font
+					(size 1.27 1.27)
+				)
+				(hide yes)
+			)
+		)
+		(property "Datasheet" ""
+			(at 151.13 111.76 0)
+			(effects
+				(font
+					(size 1.27 1.27)
+				)
+				(hide yes)
+			)
+		)
+		(property "Description" "Power symbol creates a global label with name \"GND\" , ground"
+			(at 151.13 111.76 0)
+			(effects
+				(font
+					(size 1.27 1.27)
+				)
+				(hide yes)
+			)
+		)
+		(pin "1"
+		)
+		(instances
+			(project "rs422-master"
+				(path "/a73692ab-48b2-4aab-bf01-a614ece6b97e"
+					(reference "#PWR03")
+					(unit 1)
+				)
+			)
+		)
+	)
+	(symbol
 		(lib_id "Connector:RJ45")
 		(at 184.15 95.25 180)
@@
 					(unit 1)
 				)
+			)
+		)
+	)
+	(symbol
+		(lib_id "power:+3V3")
+		(at 151.13 73.66 0)
+		(unit 1)
+		(exclude_from_sim no)
+		(in_bom yes)
+		(on_board yes)
+		(dnp no)
+		(fields_autoplaced yes)
+		(property "Reference" "#PWR02"
+			(at 151.13 77.47 0)
+			(effects
+				(font
+					(size 1.27 1.27)
+				)
+				(hide yes)
+			)
+		)
+		(property "Value" "F_5V"
+			(at 151.13 68.58 0)
+			(effects
+				(font
+					(size 1.27 1.27)
+				)
+			)
+		)
+		(property "Footprint" ""
+			(at 151.13 73.66 0)
+			(effects
+				(font
+					(size 1.27 1.27)
+				)
+				(hide yes)
+			)
+		)
+		(property "Datasheet" ""
+			(at 151.13 73.66 0)
+			(effects
+				(font
+					(size 1.27 1.27)
+				)
+				(hide yes)
+			)
+		)
+		(property "Description" "Power symbol creates a global label with name \"+3V3\""
+			(at 151.13 73.66 0)
+			(effects
+				(font
+					(size 1.27 1.27)
+				)
+				(hide yes)
+			)
+		)
+		(pin "1"
+		)
+		(instances
+			(project "rs422-master"
+				(path "/a73692ab-48b2-4aab-bf01-a614ece6b97e"
+					(reference "#PWR02")
+					(unit 1)
+				)
