File: riocore/plugins/fpga/kicad/ECP5-256/ecp5-stamp/ecp5-stamp.kicad_sch (KiCad schematic)
At the start: 24 parts, among them J1 Conn_01x06, J2 Conn_01x20, J3 Conn_01x20, J4 Conn_01x20, U10 W25Q16JVSS, U2 AMS1117-2.5, U9 ECP5U_45_CABGA256, X1 OSC_25MHz

Commit message: kicad: ecp5 tests
Parts:
- added J5, J6: Conn_02x15_Odd_Even, symbol Connector_Generic:Conn_02x15_Odd_Even
- added J7: Conn_02x15_Odd_Even, Connector_PinHeader_2.54mm:PinHeader_2x15_P2.54mm_Vertical, symbol Connector_Generic:Conn_02x15_Odd_Even
- J1: footprint Connector_PinHeader_2.54mm:PinHeader_1x06_P2.54mm_Vertical -> Connector_PinHeader_1.27mm:PinHeader_1x06_P1.27mm_Vertical
Connections:
- net A10: now also J7.17 (Pin_17)
- net A11: now also J7.19 (Pin_19)
- net A12: now also J7.21 (Pin_21)
- net A13: now also J7.23 (Pin_23)
- net A14: now also J7.25 (Pin_25)
- net A15: now also J7.27 (Pin_27)
- net A2: now also J7.2 (Pin_2)
- net A3: now also J7.4 (Pin_4)
- net A4: now also J7.6 (Pin_6)
- net A5: now also J7.8 (Pin_8)
- net A6: now also J7.10 (Pin_10)
- net A8: now also J7.13 (Pin_13)
- net A9: now also J7.15 (Pin_15)
- net B1: now also J7.1 (Pin_1)
- net B10: now also J7.18 (Pin_18)
- net B11: now also J7.20 (Pin_20)
- net B12: now also J7.22 (Pin_22)
- net B13: now also J7.24 (Pin_24)
- net B14: now also J7.26 (Pin_26)
- net B15: now also J7.28 (Pin_28)
- net B16: now also J7.29 (Pin_29)
- net B2: now also J7.3 (Pin_3)
- net B3: now also J7.5 (Pin_5)
- net B4: now also J7.7 (Pin_7)
- net B5: now also J7.9 (Pin_9)
- net B6: now also J7.11 (Pin_11)
- net B7: now also J7.12 (Pin_12)
- net B8: now also J7.14 (Pin_14)
- net B9: now also J7.16 (Pin_16)
- net JTAG.TCK: now also J1.5 (Pin_5); no longer J1.4 (Pin_4)
- net JTAG.TDO: now also J1.4 (Pin_4); no longer J1.3 (Pin_3)
- net JTAG.TMS: now also J1.3 (Pin_3); no longer J1.5 (Pin_5)
- net at J2.30 (Pin_30): now also J7.30 (Pin_30)
Other:
- moved on the sheet: J1, J2
