File: riocore/plugins/fpga/kicad/ECP5-256/ecp5-stamp/ecp5-stamp.kicad_pcb (KiCad board)
At the start: 2 copper layers, 45.2 x 51.5 mm, 24 parts, among them J1 Conn_01x06, J2 Conn_01x20, J3 Conn_01x20, J4 Conn_01x20, U10 W25Q16JVSS, U2 AMS1117-2.5, U9 ECP5U_45_CABGA256, X1 OSC_25MHz

Commit message: kicad: ecp5 tests
Parts:
- added J7: Conn_02x15_Odd_Even, Connector_PinHeader_2.54mm:PinHeader_2x15_P2.54mm_Vertical, F.Cu at (139.1, 101.5)
- J1: footprint Connector_PinHeader_2.54mm:PinHeader_1x06_P2.54mm_Vertical -> Connector_PinHeader_1.27mm:PinHeader_1x06_P1.27mm_Vertical
- moved J1 14.4 mm to (166.5, 147.5), turned to -90 degrees
Connections:
- J1 pad 3: /JTAG.TDO -> /JTAG.TMS
- J1 pad 4: /JTAG.TCK -> /JTAG.TDO
- J1 pad 5: /JTAG.TMS -> /JTAG.TCK
- J2 pad 30: unconnected-(J2-Pin_30-Pad30) -> Net-(J2-Pin_30)
Routing:
- net +3V3: track 87.6 -> 104.2 mm
- net /JTAG.TDI: track 11.4 -> 23.0 mm
- net /JTAG.TDO: track 17.0 -> 26.0 mm
- net Net-(J2-Pin_30): track 0.00 -> 6.69 mm
- net B12: track 14.3 -> 21.0 mm
- net B15: track 17.3 -> 24.0 mm
- net B14: track 15.7 -> 22.4 mm
- net B13: track 15.0 -> 21.7 mm
- net B11: track 13.6 -> 20.3 mm
- net B10: track 12.9 -> 19.6 mm
- net B8: track 12.9 -> 19.6 mm
- net B9: track 12.4 -> 19.0 mm
- net A2: track 16.7 -> 23.3 mm
- net B7: track 13.4 -> 20.0 mm
- net A3: track 15.2 -> 21.8 mm
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Other:
- board size 45.2 x 51.5 mm -> 52.5 x 57.6 mm

Commit message: kicad: ecp5 tests
Parts:
- moved C54 5.69 mm to (150.1, 134.9), turned to -90 degrees
Routing:
- net +3V3: track 104.2 -> 203.8 mm, vias 13 -> 22
- net P12: track 27.3 -> 24.7 mm
- net T14: track 21.9 -> 19.3 mm
- net R12: track 27.8 -> 25.3 mm
- net R13: track 25.0 -> 22.5 mm
- net P13: track 24.5 -> 22.1 mm
- net R14: track 21.4 -> 19.3 mm
- net R15: track 18.2 -> 20.2 mm
- net T15: track 19.0 -> 17.3 mm
- net G2: track 14.7 -> 16.4 mm
- net R16: track 18.1 -> 19.7 mm
- net G1: track 14.5 -> 16.0 mm
- net P15: track 16.3 -> 17.6 mm
- net H2: track 14.8 -> 15.8 mm
- net M1: track 12.8 -> 13.8 mm
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